File: disposable_heroes/Kicad_relesSR/VISIR_Lei_Ohm/VISIR_Lei_Ohm.kicad_sch_V8.kicad_sch (KiCad schematic)
At the start: 31 parts, among them J1 Raspberry PI5, J2 Fonte dc, J3 Fonte 12V, J4 Fonte 5V, J5 Ext_OUT_PI, J6 Ext_OUT_PI, J7 Ext_OUT_PI, J8 Ext_OUT_PI, K1 3572-1220-123, K2 3572-1220-123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

Commit message: massive update from laptop to PC
Parts:
- removed H1, H2, H3, H4: MountingHole, MountingHole:MountingHole_3.2mm_M3, symbol Mechanical:MountingHole
- removed J5, J6, J7, J8: Ext_OUT_PI, Connector_PinHeader_2.54mm:PinHeader_1x20_P2.54mm_Vertical, symbol Connector:Conn_01x20_Pin
- J1: footprint Connector_PinHeader_2.54mm:PinHeader_2x20_P2.54mm_Vertical -> Connector_PinSocket_2.54mm:PinSocket_2x20_P2.54mm_Vertical
- J2, J3, J4: footprint Connector_PinHeader_2.54mm:PinHeader_1x02_P2.54mm_Vertical -> Connector_PinSocket_2.54mm:PinSocket_1x02_P2.54mm_Vertical
Connections:
- net GND: no longer J1.30 (GND)
- no-connect marks 0 -> 2
Other:
- note added: "Relé K9 confere mais versatilidade, já que pode tornar o ramo do Amperímetro "independente""
- moved on the sheet: J1
