File: disposable_heroes/Kicad_relesSR/VISIR_Lei_Ohm/VISIR_Lei_Ohm.kicad_sch (KiCad schematic)
At the start: 31 parts, among them J1 Raspberry PI5, J2 Fonte dc, J3 Fonte 12V, J4 Fonte 5V, J5 Ext_OUT_PI, J6 Ext_OUT_PI, J7 Ext_OUT_PI, J8 Ext_OUT_PI, K1 3572-1220-123, K2 3572-1220-123, K3 3572-1220-123, K4 3570-1331-123, K5 3570-1331-123, K6 3570-1331-123, K7 3570-1331-123, K8 3570-1331-123, U1 74HC595N_112, U2 ULN2003, U3 ULN2003, U4 74HC595N_112

Commit message: update kicad meia onda
Parts:
- removed J4: Fonte 5V, Connector_PinHeader_2.54mm:PinHeader_1x02_P2.54mm_Vertical, symbol Connector:Conn_01x02_Pin
Connections:
- net +5V is gone; now on net 5VPower1: C1.1, C2.1, U1.16 (VCC), U4.16 (VCC)
- net 5VPower1: now reaches J1.2 (5VPower1), J5.20 (Pin_20), J6.20 (Pin_20)

Commit message: update kicad meiaonda e ohm
Parts:
- removed C2: 0.1uF, Capacitor_THT:C_Disc_D5.0mm_W2.5mm_P2.50mm, symbol Device:C
- removed U4: 74HC595N_112, Package_DIP:DIP-16_W10.16mm, symbol 74HC595N:74HC595N_112
- added J10: Amperimetro+, Connector_PinHeader_2.54mm:PinHeader_1x03_P2.54mm_Vertical, symbol Connector:Conn_01x03_Pin
- added J11: Amperimetro-, Connector_PinHeader_2.54mm:PinHeader_1x03_P2.54mm_Vertical, symbol Connector:Conn_01x03_Pin
- added J4: Voltimetro+, Connector_PinHeader_2.54mm:PinHeader_1x03_P2.54mm_Vertical, symbol Connector:Conn_01x03_Pin
- added J9: Voltimetro-, Connector_PinHeader_2.54mm:PinHeader_1x03_P2.54mm_Vertical, symbol Connector:Conn_01x03_Pin
- J2: value Fonte dc -> Fonte dc_VB
Connections:
- net C: now also J11.1 (Pin_1), J11.2 (Pin_2), J11.3 (Pin_3), J9.1 (Pin_1), J9.2 (Pin_2), J9.3 (Pin_3)
- net GND: no longer J1.14 (GND), J1.20 (GND), J1.25 (GND), J1.30 (GND), J1.34 (GROUND), J1.39 (GND), J1.6 (GND), J5.11 (Pin_11), J5.14 (Pin_14), J5.18 (Pin_18), J5.4 (Pin_4), J5.6 (Pin_6), J6.11 (Pin_11), J6.14 (Pin_14), J6.18 (Pin_18), J6.4 (Pin_4), J6.6 (Pin_6), J7.13 (Pin_13), J7.20 (Pin_20), J8.13 (Pin_13), J8.20 (Pin_20)
- net at K5.4, MES1.2 (+): now also J4.1 (Pin_1), J4.2 (Pin_2), J4.3 (Pin_3)
- net at K6.4, MES3.2 (+): now also J10.1 (Pin_1), J10.2 (Pin_2), J10.3 (Pin_3)
- net SER2: no longer names the net of U1.9 (Q7_2)
- new net GND1: J1.25 (GND), J7.13 (Pin_13), J8.13 (Pin_13)
- new net GND2: J1.39 (GND), J7.20 (Pin_20), J8.20 (Pin_20)
- new net GND3: J1.6 (GND), J5.18 (Pin_18), J6.18 (Pin_18)
- new net GND4: J1.14 (GND), J5.14 (Pin_14), J6.14 (Pin_14)
- new net GND5: J1.20 (GND), J5.11 (Pin_11), J6.11 (Pin_11)
- new net GND6: J1.30 (GND), J5.6 (Pin_6), J6.6 (Pin_6)
- new net GND7: J1.34 (GROUND), J5.4 (Pin_4), J6.4 (Pin_4)
Other:
- moved on the sheet: U3
