File: disposable_heroes/Kicad_relesSR/VISIR_Lei_Ohm/VISIR_Lei_Ohm.kicad_sch (KiCad schematic)
At the start: 30 parts, among them J1 Raspberry PI5, J10 Amperimetro+, J11 Amperimetro-, J4 Voltimetro+, J5 Ext_OUT_PI, J6 Ext_OUT_PI, J7 Ext_OUT_PI, J8 Ext_OUT_PI, J9 Voltimetro-, K1 3572-1220-123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

Commit message: update - boards done
Parts:
- added J2: PI_config, Connector_PinSocket_2.54mm:PinSocket_1x06_P2.54mm_Vertical, symbol Connector:Conn_01x06_Socket
- added J3: Power Sources, Connector_PinSocket_2.54mm:PinSocket_1x06_P2.54mm_Vertical, symbol Connector:Conn_01x06_Socket
Connections:
- net 12V: now also J3.1 (Pin_1)
- net 5V: now also J3.2 (Pin_2)
- net 5V_{VB}: now also J3.3 (Pin_3)
- net GND: now also J3.4 (Pin_4)
- net ~{SRCLR}_{filters}: now reaches J1.23 (GPIO11/SCLK), J7.12 (Pin_12), J8.12 (Pin_12)
- net ~{SRCLR}_{filters}: now also J2.2 (Pin_2)
- net SRCLK_{filters}: now reaches J1.7 (GPIO4/GPCLK0), J7.4 (Pin_4), J8.4 (Pin_4)
- net SRCLK_{filters}: now also J2.1 (Pin_1)
- net RCLK_{filters}: now reaches J1.11 (GPIO17), J7.6 (Pin_6), J8.6 (Pin_6)
- net RCLK_{filters}: now also J2.3 (Pin_3)
- net SER_{filters}: now reaches J1.13 (GPIO27), J7.7 (Pin_7), J8.7 (Pin_7)
- net SER_{filters}: now also J2.5 (Pin_5)
- net ~{OE}_{filters}: now reaches J1.15 (GPIO22), J7.8 (Pin_8), J8.8 (Pin_8)
- net ~{OE}_{filters}: now also J2.4 (Pin_4)
- new net transf+: J3.5 (Pin_5)
- new net transf-: J3.6 (Pin_6)
Other:
- moved on the sheet: H1, H2, H3, H4

Commit message: update kicad files
Other:
- company: (none) -> ISEP
- title: (none) -> LaRE - Rectificação meia onda
- moved on the sheet: C1, H1, H2, H3, H4, J1, J10, J11, J2, J3, J4, J5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
