File: disposable_heroes/Kicad_relesSR/VISIR_Lei_Ohm/VISIR_Lei_Ohm.kicad_pcb (KiCad board)
At the start: 2 copper layers, 17 parts, among them J1 Raspberry PI5, J2 Fonte 5V, K1 3572-1220-123, K2 3572-1220-123, K3 3572-1220-123, K4 3570-1331-123, K5 3570-1331-123, K6 3570-1331-123, K7 3570-1331-123, K8 3570-1331-123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

Commit message: update kicad
Parts:
- removed MES2: Ammeter_DC, Connector_PinHeader_2.54mm:PinHeader_1x02_P2.54mm_Vertical_SMD_Pin1Left
- added C1: 0.1uF, Capacitor_THT:C_Disc_D5.0mm_W2.5mm_P2.50mm, F.Cu at (133.2, 64.4)
- added C2: 0.1uF, Capacitor_THT:C_Disc_D5.0mm_W2.5mm_P2.50mm, F.Cu at (133.2, 68.5)
- added J3: Fonte 12V, Connector_PinSocket_2.54mm:PinSocket_1x02_P2.54mm_Vertical, F.Cu at (200.1, 76.2)
- added J4: Fonte 5V, Connector_PinSocket_2.54mm:PinSocket_1x02_P2.54mm_Vertical, F.Cu at (200.1, 71.7)
- added MES3: Ammeter_DC, Connector_PinHeader_2.54mm:PinHeader_1x02_P2.54mm_Vertical, F.Cu at (200.1, 85.5)
- added U3: ULN2003, Package_DIP:DIP-16_W10.16mm, F.Cu at (152.2, 73.8)
- added U4: 74HC595N_112, Package_DIP:DIP-16_W10.16mm, F.Cu at (165.6, 73.8)
- J2: value Fonte 5V -> Fonte dc
- K1, K2, K3: footprint 3572-1220-053:RELAY8_3572-1220-053_COM -> rele_DPST_tese:RELAY8_3572-1220-053_COM
- K4, K5, K6, K7, K8: footprint 3570-1220-123:SIP_3570-1331_COM -> rele_SPST_tese:SIP_3570-1331_COM
- moved R3 160.3 mm to (191.5, 88.4), turned to 90 degrees
- moved R2 156.3 mm to (187.5, 88.4), turned to 90 degrees
- moved R1 152.5 mm to (183.4, 88.4), turned to 90 degrees
- moved K8 136.0 mm to (167.6, 58.3), turned to 90 degrees
- moved J1 134.8 mm to (175.0, 108.3), turned to -90 degrees
- moved K7 128.4 mm to (158.7, 43.1), turned to -90 degrees
- moved K1 125.0 mm to (176.8, 43.1)
- moved K2 125.0 mm to (187.3, 43.1)
- moved K3 125.0 mm to (197.9, 43.1)
- moved K6 116.0 mm to (147.2, 43.1), turned to -90 degrees
- moved MES1 115.6 mm to (200.1, 90.2), turned to 90 degrees
- moved K5 104.5 mm to (136.8, 58.3), turned to 90 degrees
- moved J2 96.9 mm to (200.1, 80.8)
- moved K4 96.1 mm to (127.8, 58.3), turned to 90 degrees
- moved U1 74.1 mm to (125.5, 73.8)
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Connections:
- net /I_{1} renamed /I_{11}
- net /I_{2} renamed /I_{12}
- net /I_{3} renamed /I_{13}
- net /I_{4} renamed /I_{14}
- net /I_{5} renamed /I_{15}
- net /I_{6} renamed /I_{16}
- net /I_{7} renamed /I_{17}
- net /O_{1} renamed /O_{11}
- net /O_{2} renamed /O_{12}
- net /O_{3} renamed /O_{13}
- net /O_{4} renamed /O_{14}
- net /O_{5} renamed /O_{15}
- J1 pad 29: unconnected-(J1-GPIO5-Pad29) -> /SER1
- J1 pad 31: unconnected-(J1-GPIO6-Pad31) -> /RCLK
- J1 pad 33: unconnected-(J1-GPIO13/PWM1-Pad33) -> /SRCLK
- J1 pad 35: unconnected-(J1-GPIO19/PCM_FS-Pad35) -> /~{OE}
- J1 pad 37: unconnected-(J1-GPIO26-Pad37) -> /~{SRCLR}
- J2 pad 1: +5V -> VCC
- J2 pad 2: GND -> D
- K3 pad 1: GND -> B
- K4 pad 1: +5V -> VCC
- K5 pad 4: B -> Net-(MES1-+)
- K6 pad 1: Net-(MES2-+) -> B
- K6 pad 2: Net-(MES2-+) -> +12V
- K6 pad 3: /O6 -> /O_{16}
- K6 pad 4: B -> Net-(MES3-+)
- K7 pad 1: Net-(MES2--) -> C
- K7 pad 3: /O7 -> /O_{17}
- K8 pad 3: /O8 -> /O_{21}
- K8 pad 4: GND -> C
- MES1 pad 1: GND -> C
- MES1 pad 2: A -> Net-(MES1-+)
- U1 pad 10: /~{MR} -> /~{SRCLR}
- U1 pad 11: /SH_CP -> /SRCLK
- U1 pad 12: /ST_CP -> /RCLK
- U1 pad 14: /DS -> /SER1
- U1 pad 7: unconnected-(U1-Q7-Pad7) -> /I_{21}
- U1 pad 9: unconnected-(U1-Q7_2-Pad9) -> /SER2
- U2 pad 10: /O_{7} -> /O_{17}
- U2 pad 11: /O_{6} -> /O_{16}
Routing:
- net GND: track 0.00 -> 248.5 mm
- net +12V: track 0.00 -> 192.0 mm
- net C: track 0.00 -> 165.3 mm
- net A: track 0.00 -> 114.8 mm
- net B: track 0.00 -> 97.7 mm
- net Net-(MES1-+): track 0.00 -> 97.4 mm
- net /~{SRCLR}: track 0.00 -> 87.9 mm, vias 0 -> 1
- net +5V: track 0.00 -> 86.5 mm
- net VCC: track 0.00 -> 84.6 mm, vias 0 -> 1
- net /SRCLK: track 0.00 -> 82.0 mm
- net /I_{21}: track 0.00 -> 78.5 mm
- net Net-(K3-Pad8): track 0.00 -> 78.2 mm
- net /RCLK: track 0.00 -> 71.9 mm, vias 0 -> 1
- net /~{OE}: track 0.00 -> 69.8 mm
- net Net-(MES3-+): track 0.00 -> 68.0 mm, vias 0 -> 1
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
Commit message: massive update from laptop to PC
Parts:
- added H1: MountingHole, MountingHole:MountingHole_3.2mm_M3, F.Cu at (210.9, 35.6)
- added H2: MountingHole, MountingHole:MountingHole_3.2mm_M3, F.Cu at (125.7, 35.5)
- added H3: MountingHole, MountingHole:MountingHole_3.2mm_M3, F.Cu at (126.0, 115.8)
- added H4: MountingHole, MountingHole:MountingHole_3.2mm_M3, F.Cu at (210.7, 115.8)
- added J5: Ext_OUT_PI, Connector_PinHeader_2.54mm:PinHeader_1x20_P2.54mm_Vertical, F.Cu at (142.0, 113.9)
- added J6: Ext_OUT_PI, Connector_PinHeader_2.54mm:PinHeader_1x20_P2.54mm_Vertical, F.Cu at (141.9, 117.8)
- added J7: Ext_OUT_PI, Connector_PinHeader_2.54mm:PinHeader_1x20_P2.54mm_Vertical, F.Cu at (190.3, 101.8)
- added J8: Ext_OUT_PI, Connector_PinHeader_2.54mm:PinHeader_1x20_P2.54mm_Vertical, F.Cu at (190.2, 98.0)
- J1: footprint Connector_PinSocket_2.54mm:PinSocket_2x20_P2.54mm_Vertical -> Connector_PinHeader_2.54mm:PinHeader_2x20_P2.54mm_Vertical
- J2, J3, J4: footprint Connector_PinSocket_2.54mm:PinSocket_1x02_P2.54mm_Vertical -> Connector_PinHeader_2.54mm:PinHeader_1x02_P2.54mm_Vertical
- moved J1 15.3 mm to (190.2, 106.6)
Connections:
- J1 pad 1: unconnected-(J1-3V3Power-Pad1) -> Net-(J1-3V3Power)
- J1 pad 10: unconnected-(J1-GPIO15/RXD-Pad10) -> Net-(J1-GPIO15/RXD)
- J1 pad 11: unconnected-(J1-GPIO17-Pad11) -> Net-(J1-GPIO17)
- J1 pad 12: unconnected-(J1-GPIO18/PCM_CLK-Pad12) -> Net-(J1-GPIO18/PCM_CLK)
- J1 pad 13: unconnected-(J1-GPIO27-Pad13) -> Net-(J1-GPIO27)
- J1 pad 15: unconnected-(J1-GPIO22-Pad15) -> Net-(J1-GPIO22)
- J1 pad 16: unconnected-(J1-GPIO23-Pad16) -> Net-(J1-GPIO23)
- J1 pad 17: unconnected-(J1-3v3Power-Pad17) -> Net-(J1-3v3Power)
- J1 pad 18: unconnected-(J1-GPIO24-Pad18) -> Net-(J1-GPIO24)
- J1 pad 19: unconnected-(J1-GPIO10/MOSI-Pad19) -> Net-(J1-GPIO10/MOSI)
- J1 pad 2: unconnected-(J1-5VPower-Pad2) -> Net-(J5-Pin_20)
- J1 pad 21: unconnected-(J1-GPIO9/MISO-Pad21) -> Net-(J1-GPIO9/MISO)
- J1 pad 22: unconnected-(J1-GPIO25-Pad22) -> Net-(J1-GPIO25)
- J1 pad 23: unconnected-(J1-GPIO11/SCLK-Pad23) -> Net-(J1-GPIO11/SCLK)
- J1 pad 24: unconnected-(J1-GPIO8/CE0-Pad24) -> Net-(J1-GPIO8/CE0)
- J1 pad 26: unconnected-(J1-GPIO7/CE1-Pad26) -> Net-(J1-GPIO7/CE1)
- J1 pad 27: unconnected-(J1-GPIO0/ID_SD-Pad27) -> Net-(J1-GPIO0/ID_SD)
- J1 pad 28: unconnected-(J1-GPIO1/ID_SC-Pad28) -> Net-(J1-GPIO1/ID_SC)
- J1 pad 3: unconnected-(J1-GPIO2/SDA-Pad3) -> Net-(J1-GPIO2/SDA)
- J1 pad 30: unconnected-(J1-GND-Pad30) -> GND
- J1 pad 32: unconnected-(J1-GPIO12/PWM0-Pad32) -> Net-(J1-GPIO12/PWM0)
- J1 pad 36: unconnected-(J1-GPIO16-Pad36) -> Net-(J1-GPIO16)
- J1 pad 38: unconnected-(J1-GPIO20/PCM_DIN-Pad38) -> Net-(J1-GPIO20/PCM_DIN)
- J1 pad 4: unconnected-(J1-5VPower-Pad4) -> Net-(J5-Pin_19)
- J1 pad 40: unconnected-(J1-GPIO21/PCM_DOUT-Pad40) -> Net-(J1-GPIO21/PCM_DOUT)
- J1 pad 5: unconnected-(J1-GPIO3/SCL-Pad5) -> Net-(J1-GPIO3/SCL)
- J1 pad 7: unconnected-(J1-GPIO4/GPCLK0-Pad7) -> Net-(J1-GPIO4/GPCLK0)
- J1 pad 8: unconnected-(J1-GPIO14/TXD-Pad8) -> Net-(J1-GPIO14/TXD)
Routing:
- net C: track 165.3 -> 80.3 mm
- net /I_{21}: track 78.5 -> 34.9 mm
- net Net-(J1-3v3Power): track 0.00 -> 39.0 mm
- net Net-(K3-Pad8): track 78.2 -> 41.7 mm
- net B: track 97.7 -> 67.5 mm
- net /~{SRCLR}: track 87.9 -> 61.1 mm, vias 1 -> 0
- net +12V: track 192.0 -> 166.3 mm
- net /SRCLK: track 82.0 -> 61.8 mm
- net /SER2: track 65.4 -> 45.5 mm, vias 2 -> 0
- net Net-(MES3-+): track 68.0 -> 87.1 mm, vias 1 -> 0
- net VCC: track 84.6 -> 103.2 mm, vias 1 -> 0
- net A: track 114.8 -> 96.2 mm
- net Net-(MES1-+): track 97.4 -> 111.1 mm
- net GND: track 248.5 -> 261.1 mm
- net Net-(J1-GPIO2/SDA): track 0.00 -> 9.21 mm
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- added copper zone on B.Cu, net GND
- added copper zone on F.Cu, net GND

Commit message: update kicad meia onda
Parts:
- removed J4: Fonte 5V, Connector_PinHeader_2.54mm:PinHeader_1x02_P2.54mm_Vertical
Connections:
- C1 pad 1: +5V -> /5VPower1
- C2 pad 1: +5V -> /5VPower1
- J1 pad 2: Net-(J5-Pin_20) -> /5VPower1
- J5 pad 20: Net-(J5-Pin_20) -> /5VPower1
- J6 pad 20: Net-(J5-Pin_20) -> /5VPower1
- U1 pad 16: +5V -> /5VPower1
- U4 pad 16: +5V -> /5VPower1
Routing:
- net /5VPower1: track 0.00 -> 104.1 mm
- net +5V: track 80.4 -> 0.00 mm, vias 1 -> 0
- net Net-(J1-3v3Power2): track 39.0 -> 8.62 mm
- net /SER1: track 37.6 -> 67.7 mm
- net /~{OE}: track 66.5 -> 92.4 mm
- net /RCLK: track 80.5 -> 68.0 mm
- net Net-(J5-Pin_20): track 8.77 -> 0.00 mm
- net Net-(J1-3V3Power1): track 0.00 -> 8.62 mm
- net Net-(K3-Pad8): track 41.7 -> 35.9 mm
- net C: track 80.3 -> 85.8 mm
- net /O_{13}: track 65.1 -> 59.9 mm
- net /O_{12}: track 46.8 -> 51.5 mm
- net +12V: track 166.3 -> 170.9 mm
- net /I_{17}: track 18.9 -> 14.4 mm
- net /~{SRCLR}: track 61.1 -> 57.0 mm
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- removed copper zone on B.Cu, net GND
- removed copper zone on F.Cu, net GND

Commit message: update kicad meiaonda e ohm
Parts:
- removed C2: 0.1uF, Capacitor_THT:C_Disc_D5.0mm_W2.5mm_P2.50mm
- removed U4: 74HC595N_112, Package_DIP:DIP-16_W10.16mm
- added J10: Amperimetro+, Connector_PinHeader_2.54mm:PinHeader_1x03_P2.54mm_Vertical, F.Cu at (196.2, 84.8)
- added J11: Amperimetro-, Connector_PinHeader_2.54mm:PinHeader_1x03_P2.54mm_Vertical, F.Cu at (199.9, 84.8)
- added J4: Voltimetro+, Connector_PinHeader_2.54mm:PinHeader_1x03_P2.54mm_Vertical, F.Cu at (207.6, 84.8)
- added J9: Voltimetro-, Connector_PinHeader_2.54mm:PinHeader_1x03_P2.54mm_Vertical, F.Cu at (211.4, 84.9)
- J2: value Fonte dc -> Fonte dc_VB
- moved MES1 14.8 mm to (210.7, 79.8), turned to -90 degrees
- moved R1 11.2 mm to (172.2, 88.3)
- moved R2 11.2 mm to (176.2, 88.3)
- moved R3 11.2 mm to (180.3, 88.3)
- moved J3 9.65 mm to (196.6, 67.2)
- moved J2 9.37 mm to (196.5, 72.2)
- moved MES3 5.70 mm to (199.2, 79.9), turned to -90 degrees
Connections:
- J1 pad 14: GND -> GND4
- J1 pad 20: GND -> GND5
- J1 pad 25: GND -> GND1
- J1 pad 30: GND -> GND6
- J1 pad 34: GND -> GND7
- J1 pad 39: GND -> GND2
- J1 pad 6: GND -> GND3
- J5 pad 11: GND -> GND5
- J5 pad 14: GND -> GND4
- J5 pad 18: GND -> GND3
- J5 pad 4: GND -> GND7
- J5 pad 6: GND -> GND6
- J6 pad 11: GND -> GND5
- J6 pad 14: GND -> GND4
- J6 pad 18: GND -> GND3
- J6 pad 4: GND -> GND7
- J6 pad 6: GND -> GND6
- J7 pad 13: GND -> GND1
- J7 pad 20: GND -> GND2
- J8 pad 13: GND -> GND1
- J8 pad 20: GND -> GND2
- U1 pad 9: /SER2 -> unconnected-(U1-Q7_2-Pad9)
Routing:
- net GND: track 258.0 -> 158.9 mm
- net /~{OE}: track 92.4 -> 44.8 mm
- net /SER2: track 45.5 -> 0.00 mm
- net /RCLK: track 68.0 -> 31.3 mm
- net /~{SRCLR}: track 57.0 -> 23.3 mm
- net /SRCLK: track 62.5 -> 29.4 mm, vias 0 -> 1
- net C: track 85.8 -> 115.9 mm
- net /SER1: track 67.7 -> 37.9 mm
- net /I_{22}: track 24.4 -> 0.00 mm
- net +12V: track 170.9 -> 154.7 mm
- net VCC: track 103.3 -> 92.9 mm
- net GND6: track 0.00 -> 8.77 mm
- net GND5: track 0.00 -> 8.77 mm
- net GND4: track 0.00 -> 8.77 mm
- net GND7: track 0.00 -> 8.77 mm
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- added copper zone on B.Cu, net GND
- added copper zone on F.Cu, net GND
Other:
- board outline added: 95.3 x 90.1 mm

Commit message: update kicad
Parts:
- J3: value Fonte 12V -> 12V; footprint Connector_PinHeader_2.54mm:PinHeader_1x02_P2.54mm_Vertical -> Connector_PinHeader_2.54mm:PinHeader_1x06_P2.54mm_Vertical
Connections:
- J3 pad 1: +12V -> /12V
- J3 pad 2: GND -> /12V
- K1 pad 2: +12V -> /12V
- K2 pad 2: +12V -> /12V
- K3 pad 2: +12V -> /12V
- K4 pad 2: +12V -> unconnected-(K4-Pad2)
- K5 pad 2: +12V -> /12V
- K6 pad 2: +12V -> /12V
- K7 pad 2: +12V -> /12V
- K8 pad 2: +12V -> /12V
- U2 pad 9: +12V -> /12V
- U3 pad 9: +12V -> /12V
Routing:
- net GND: track 158.9 -> 0.00 mm
- net +12V: track 154.7 -> 0.00 mm
- net C: track 115.9 -> 0.00 mm
- net Net-(J4-Pin_1): track 114.9 -> 0.00 mm
- net /5VPower1: track 102.6 -> 0.00 mm
- net A: track 96.1 -> 0.00 mm
- net VCC: track 92.9 -> 0.00 mm
- net Net-(J10-Pin_1): track 90.0 -> 0.00 mm
- net B: track 67.4 -> 0.00 mm
- net /O_{13}: track 58.4 -> 0.00 mm
- net /O_{12}: track 46.8 -> 0.00 mm
- net /I_{21}: track 46.2 -> 0.00 mm
- net /~{OE}: track 44.8 -> 0.00 mm
- net /O_{14}: track 42.3 -> 0.00 mm
- net /O_{15}: track 42.0 -> 0.00 mm
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- removed copper zone on B.Cu, net GND
- removed copper zone on F.Cu, net GND

Commit message: update - boards done
Parts:
- J2: value Fonte dc_VB -> Power Sources; footprint Connector_PinHeader_2.54mm:PinHeader_1x02_P2.54mm_Vertical -> Connector_PinSocket_2.54mm:PinSocket_1x06_P2.54mm_Vertical
- J3: value 12V -> PI_config; footprint Connector_PinHeader_2.54mm:PinHeader_1x06_P2.54mm_Vertical -> Connector_PinSocket_2.54mm:PinSocket_1x06_P2.54mm_Vertical
- moved H2 117.5 mm to (211.5, 115.7)
- moved H4 115.0 mm to (125.8, 38.2)
- moved J2 53.4 mm to (155.3, 38.2), turned to -90 degrees
- moved J3 35.7 mm to (175.9, 38.2), turned to -90 degrees
- moved J10 9.25 mm to (188.0, 80.4)
- moved J9 9.25 mm to (203.2, 80.5)
- moved MES3 9.25 mm to (191.1, 75.5)
- moved J11 9.25 mm to (191.8, 80.5)
- moved J4 9.25 mm to (199.4, 80.5)
- moved MES1 9.25 mm to (202.6, 75.5)
- moved K3 6.08 mm to (202.7, 46.8)
- moved C1 5.90 mm to (135.8, 69.7)
- moved K2 4.23 mm to (189.6, 46.7)
- moved K7 4.06 mm to (156.8, 46.7)
- moved H3 3.85 mm to (125.8, 111.9)
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Connections:
- C1 pad 1: /5VPower1 -> /5V
- J1 pad 11: Net-(J1-GPIO17) -> /RCLK_{filters}
- J1 pad 13: Net-(J1-GPIO27) -> /SER_{filters}
- J1 pad 15: Net-(J1-GPIO22) -> /~{OE}_{filters}
- J1 pad 23: Net-(J1-GPIO11/SCLK) -> /~{SRCLR}_{filters}
- J1 pad 7: Net-(J1-GPIO4/GPCLK0) -> /SRCLK_{filters}
- J2 pad 1: VCC -> /12V
- J2 pad 2: D -> /5V
- J3 pad 1: /12V -> /SRCLK_{filters}
- J3 pad 2: /12V -> /~{SRCLR}_{filters}
- J3 pad 3: /12V -> /RCLK_{filters}
- J3 pad 4: /12V -> /~{OE}_{filters}
- J3 pad 5: /12V -> /SER_{filters}
- J3 pad 6: /12V -> unconnected-(J3-Pin_6-Pad6)
- J7 pad 12: Net-(J1-GPIO11/SCLK) -> /~{SRCLR}_{filters}
- J7 pad 4: Net-(J1-GPIO4/GPCLK0) -> /SRCLK_{filters}
- J7 pad 6: Net-(J1-GPIO17) -> /RCLK_{filters}
- J7 pad 7: Net-(J1-GPIO27) -> /SER_{filters}
- J7 pad 8: Net-(J1-GPIO22) -> /~{OE}_{filters}
- J8 pad 12: Net-(J1-GPIO11/SCLK) -> /~{SRCLR}_{filters}
- J8 pad 4: Net-(J1-GPIO4/GPCLK0) -> /SRCLK_{filters}
- J8 pad 6: Net-(J1-GPIO17) -> /RCLK_{filters}
- J8 pad 7: Net-(J1-GPIO27) -> /SER_{filters}
- J8 pad 8: Net-(J1-GPIO22) -> /~{OE}_{filters}
- K4 pad 1: VCC -> /5V_{VB}
- K4 pad 2: unconnected-(K4-Pad2) -> /12V
- U1 pad 16: /5VPower1 -> /5V
Routing:
- net GND: track 0.00 -> 167.1 mm
- net /12V: track 0.00 -> 148.4 mm
- net /I_{21}: track 0.00 -> 132.9 mm
- net A: track 0.00 -> 103.9 mm
- net Net-(J4-Pin_1): track 0.00 -> 102.9 mm
- net C: track 0.00 -> 87.7 mm, vias 0 -> 1
- net /~{SRCLR}_{filters}: track 0.00 -> 80.4 mm
- net /SER_{filters}: track 0.00 -> 78.6 mm
- net B: track 0.00 -> 77.7 mm
- net /~{OE}_{filters}: track 0.00 -> 73.0 mm
- net /RCLK_{filters}: track 0.00 -> 71.2 mm
- net /SRCLK_{filters}: track 0.00 -> 71.2 mm
- net Net-(J10-Pin_1): track 0.00 -> 63.4 mm, vias 0 -> 1
- net /O_{13}: track 0.00 -> 61.7 mm
- net /O_{14}: track 0.00 -> 53.3 mm
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- added copper zone on B.Cu, net GND
- added copper zone on F.Cu, net GND
Other:
- board size 95.3 x 90.1 mm -> 96 x 90.5 mm
- board text added: "LaRE - Lei de OHM"

Commit message: updates finais
Parts:
- moved MES3 24.2 mm to (211.9, 88.0), turned to 180 degrees
- moved J10 19.5 mm to (206.9, 84.9), turned to -90 degrees
- moved J11 17.2 mm to (206.9, 88.6), turned to -90 degrees
- moved J4 10.5 mm to (207.1, 73.2), turned to -90 degrees
- moved MES1 9.56 mm to (212.1, 76.4), turned to 180 degrees
- moved J9 5.17 mm to (207.1, 77.0), turned to -90 degrees
- moved J6 1.11 mm to (142.0, 116.7)
- moved J5 0.88 mm to (142.0, 113.0)
- moved J1 0.30 mm to (190.2, 106.3)
Routing:
- net Net-(J10-Pin_1): track 63.4 -> 80.0 mm
- net C: track 87.7 -> 102.5 mm
- net Net-(J4-Pin_1): track 102.9 -> 106.2 mm
- net GND3: track 8.77 -> 10.1 mm
- net Net-(K3-Pad8): track 41.9 -> 40.9 mm
- net Net-(J1-GPIO20/PCM_DIN): track 8.77 -> 7.95 mm
- net Net-(J1-GPIO21/PCM_DOUT): track 8.77 -> 7.95 mm
- net Net-(J1-GPIO15/RXD): track 8.77 -> 7.97 mm
- net Net-(J1-GPIO16): track 8.77 -> 8.01 mm
- net GND7: track 8.77 -> 8.01 mm
- net GND5: track 8.77 -> 8.01 mm
- net GND4: track 8.77 -> 8.01 mm
- net Net-(J1-GPIO8/CE0): track 8.77 -> 8.01 mm
- net Net-(J1-GPIO7/CE1): track 8.77 -> 8.01 mm
- net Net-(J1-GPIO25): track 8.77 -> 8.01 mm
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