File: disposable_heroes/Kicad_relesSR/meiaonda/_autosave-meiaonda.kicad_sch (KiCad schematic)
At the start: 43 parts, among them J1 Vgen, J10 Transformer, J2 Fonte 12V, J3 Fonte 5V - PI5, J4 GPIO11, J5 GPIO26, J6 GPIO6, J7 GPIO13, J8 GPIO5, K1 3572-1220-123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

Commit message: update
Other:
- note added: "K1"
- note added: "K2"
- note added: "K3"
Changed lines of the file:
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@@
+		)
+	)
+	(text "K2"
+		(exclude_from_sim no)
+		(at 132.334 172.212 0)
+		(effects
+			(font
+				(size 1.27 1.27)
+			)
 		)
 	)
@@
 		(exclude_from_sim no)
 		(at 353.314 59.944 0)
+		(effects
+			(font
+				(size 1.27 1.27)
+			)
+		)
+	)
+	(text "K3\n"
+		(exclude_from_sim no)
+		(at 132.588 174.498 0)
 		(effects
 			(font
@@
 		(effects
 			(font
+				(size 1.27 1.27)
+			)
+		)
+	)
+	(text "K1"
+		(exclude_from_sim no)
+		(at 132.588 169.672 0)
+		(effects
+			(font
