File: disposable_heroes/Kicad_relesSR/meiaonda/meiaonda.kicad_sch (KiCad schematic)
At the start: 43 parts, among them J1 Vgen, J10 Transformer, J2 Fonte 12V, J3 Fonte 5V - PI5, J4 GPIO11, J5 GPIO26, J6 GPIO6, J7 GPIO13, J8 GPIO5, K1 3572-1220-123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

Commit message: update
Parts:
- J4: value GPIO11 -> GPIO22
- J8: value GPIO5 -> GPIO27
Other:
- note added: "K1"
- note added: "K2"
- note added: "K3"
Changed lines of the file:
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@@
+		)
+	)
+	(text "K2"
+		(exclude_from_sim no)
+		(at 132.334 172.212 0)
+		(effects
+			(font
+				(size 1.27 1.27)
+			)
 		)
 	)
@@
 		)
 	)
+	(text "K3\n"
+		(exclude_from_sim no)
+		(at 132.588 174.498 0)
+		(effects
+			(font
+				(size 1.27 1.27)
+			)
+		)
+	)
 	(text "8 relés duplos\n1 relé simples"
 		(exclude_from_sim no)
@@
 		(exclude_from_sim no)
 		(at 63.5 23.114 0)
+		(effects
+			(font
+				(size 1.27 1.27)
+			)
+		)
+	)
+	(text "K1"
+		(exclude_from_sim no)
+		(at 132.588 169.672 0)
 		(effects
 			(font
@@
 			)
 		)
-		(property "Value" "GPIO11"
+		(property "Value" "GPIO22"
 			(at 40.64 175.26 0)
 			(effects
@@
 			)
 		)
-		(property "Value" "GPIO5"
+		(property "Value" "GPIO27"
 			(at 40.132 193.04 0)
 			(effects

Commit message: update
Parts:
- J3: value Fonte 5V - PI5 -> Fonte 5V - VB
Other:
- note added: "1"
- note added: "K1 0"
- note removed: "K1"
Changed lines of the file:
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@@
 		)
 	)
-	(text "K1"
+	(text "1"
+		(exclude_from_sim no)
+		(at 103.378 168.402 0)
+		(effects
+			(font
+				(size 1.27 1.27)
+			)
+		)
+	)
+	(text "K1\n0"
 		(exclude_from_sim no)
 		(at 132.588 169.672 0)
@@
 			)
 		)
-		(property "Value" "Fonte 5V - PI5"
+		(property "Value" "Fonte 5V - VB"
 			(at 201.0156 117.4496 90)
 			(effects

Commit message: update onda completa
Parts:
- added J9: Canal 2 - V_{out}, Connector_PinHeader_2.54mm:PinHeader_1x02_P2.54mm_Vertical, symbol Connector:Conn_01x02_Pin
- added K12: 3570-1331-123, 3570-1331-123:SIP_3570-1331_COM, symbol 3570-1331-123:3570-1331-123
- J1: value Vgen -> Canal 1 - V_{in}
- renumbered K12 to K13, K13 to K14
Connections:
- net +12V: now also K12.2
- net I_{25}: now also U3.3 (Q3)
- net bypass neg: now also J9.1 (Pin_1)
- net at D2.2: now also K2.8; no longer K2.7
- net at D2.3: now also K2.7; no longer K2.1
- net at K1.1: now also F1.2, J1.2 (Pin_2), K2.14; no longer J1.1 (Pin_1)
- net at K1.8: now also J10.1 (Pin_1), K2.1, K12.4; no longer J1.2 (Pin_2)
- net at J10.2 (Pin_2): now also F1.1; no longer K2.14
- net at K4.4, K5.8, K6.8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: now also J9.2 (Pin_2)
- net O_{25}: now reaches U4.12 (O5)
- net O_{25}: now also K12.3
- new net: J1.1 (Pin_1), K12.1
Other:
- note added: "Pontas osciloscópio"
- note added: "Relé K12 necessário por causa das massas no rectificador de onda completa"
- note removed: "Gerador de sinal"
- moved on the sheet: C1, C2, C3, C4, D1, D2, F1, J1, J10, J2, J3, J4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
