File: disposable_heroes/Kicad_relesSR/meiaonda/meiaonda.kicad_sch (KiCad schematic)
At the start: 42 parts, among them J1 Canal 1 - V_{in}, J10 Gerador Sinal, J2 Transformer, J3 Power Sources, J4 GPIO22, J5 GPIO26, J6 GPIO6, J7 GPIO13, J8 GPIO27, J9 Canal 2 - V_{out}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

Commit message: update - boards done
Parts:
- removed J1: Canal 1 - V_{in}, Connector_PinHeader_2.54mm:PinHeader_1x02_P2.54mm_Vertical, symbol Connector:Conn_01x02_Socket
- removed J10: Gerador Sinal, Connector_PinHeader_2.54mm:PinHeader_1x02_P2.54mm_Vertical, symbol Connector:Conn_01x02_Pin
- removed J2: Transformer, Connector_PinHeader_2.54mm:PinHeader_1x02_P2.54mm_Vertical, symbol Connector:Conn_01x02_Pin
- removed J3: Power Sources, symbol Connector:Conn_01x04_Socket
- removed J4: GPIO22, Connector_PinHeader_2.54mm:PinHeader_1x01_P2.54mm_Vertical, symbol Connector:Conn_01x01_Pin
- removed J5: GPIO26, Connector_PinHeader_2.54mm:PinHeader_1x01_P2.54mm_Vertical, symbol Connector:Conn_01x01_Pin
- removed J6: GPIO6, Connector_PinHeader_2.54mm:PinHeader_1x01_P2.54mm_Vertical, symbol Connector:Conn_01x01_Pin
- removed J7: GPIO13, Connector_PinHeader_2.54mm:PinHeader_1x01_P2.54mm_Vertical, symbol Connector:Conn_01x01_Pin
- removed J8: GPIO27, Connector_PinHeader_2.54mm:PinHeader_1x01_P2.54mm_Vertical, symbol Connector:Conn_01x01_Pin
- removed J9: Canal 2 - V_{out}, Connector_PinHeader_2.54mm:PinHeader_1x02_P2.54mm_Vertical, symbol Connector:Conn_01x02_Pin
- added J2: PI_config, Connector_PinSocket_2.54mm:PinSocket_1x06_P2.54mm_Vertical, symbol Connector:Conn_01x06_Socket
- added J3: Power Sources, Connector_PinSocket_2.54mm:PinSocket_1x06_P2.54mm_Vertical, symbol Connector:Conn_01x06_Socket
- added J4: Signals, Connector_PinSocket_2.54mm:PinSocket_1x06_P2.54mm_Vertical, symbol Connector:Conn_01x06_Pin
Connections:
- net 12V: now also J3.1 (Pin_1)
- net 5V: now also J3.2 (Pin_2)
- net 5V_{VB}: now also J3.3 (Pin_3)
- net CH_{1}+: now also J4.1 (Pin_1), J4.3 (Pin_3); no longer K1.8, K12.1
- net GND: now also J3.4 (Pin_4)
- net v_{out}+: now also J4.5 (Pin_5)
- net v_{out}-: now also J4.6 (Pin_6); no longer K6.8
- net ~{SRCLR}_{filters}: now reaches U1.10 (~SRCLR), U3.10 (~SRCLR)
- net ~{SRCLR}_{filters}: now also J2.2 (Pin_2)
- net SRCLK_{filters}: now reaches U1.11 (SRCLK), U3.11 (SRCLK)
- net SRCLK_{filters}: now also J2.1 (Pin_1)
- net RCLK_{filters}: now reaches U1.12 (RCLK), U3.12 (RCLK)
- net RCLK_{filters}: now also J2.3 (Pin_3)
- net ~{OE}_{filters}: now reaches U1.13 (~OE), U3.13 (~OE)
- net ~{OE}_{filters}: now also J2.4 (Pin_4)
- net SER_{filters}: now reaches U1.14 (SER)
- net SER_{filters}: now also J2.5 (Pin_5)
- net transf-: now reaches K2.1
- net transf-: now also J3.6 (Pin_6)
- net transf+: now reaches F1.1
- net transf+: now also J3.5 (Pin_5)
- new net CH_{1}-: J4.2 (Pin_2), J4.4 (Pin_4), K1.8, K12.1
- no-connect marks 0 -> 1
Other:
- note removed: "1"
- note removed: "K1 0"
- note removed: "K2"
- note removed: "K3"
- note removed: "K9"
- note removed: "~8V"

Commit message: update kicad files
Other:
- note added: "Filtragem"
- note added: "Gerador de sinal"
- note removed: "Reles simples"
- company: (none) -> ISEP
- title: (none) -> LaRE - Rectificação/Filtragem
- moved on the sheet: C6, K10, K11, R3
Changed lines of the file:
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@@
 	(generator_version "8.0")
 	(paper "A3")
+	(title_block
+		(title "LaRE - Rectificação/Filtragem")
+		(date "2024-07-21")
+		(rev "Julho 2024")
+		(company "ISEP")
+	)
 	(junction
 		(at 157.48 229.87)
@@
 	)
 	(junction
-		(at 328.93 53.34)
+		(at 273.05 106.68)
 		(diameter 0)
 		(color 0 0 0 0)
@@
 	(wire
 		(pts
-			(xy 349.25 50.8) (xy 345.44 50.8)
+			(xy 293.37 104.14) (xy 289.56 104.14)
 		)
 		(stroke
@@
 	(wire
 		(pts
-			(xy 364.49 68.58) (xy 374.65 68.58)
+			(xy 308.61 121.92) (xy 318.77 121.92)
 		)
 		(stroke
@@
 	(wire
 		(pts
-			(xy 328.93 53.34) (xy 328.93 49.53)
+			(xy 273.05 106.68) (xy 273.05 102.87)
 		)
 		(stroke
@@
 	(wire
 		(pts
-			(xy 345.44 50.8) (xy 345.44 68.58)
+			(xy 289.56 104.14) (xy 289.56 121.92)
 		)
 		(stroke
@@
 	(wire
 		(pts
-			(xy 374.65 58.42) (xy 374.65 60.96)
+			(xy 318.77 111.76) (xy 318.77 114.3)
 		)
 		(stroke
@@
 	(wire
 		(pts
-			(xy 365.76 50.8) (xy 374.65 50.8)
+			(xy 309.88 104.14) (xy 318.77 104.14)
 		)
 		(stroke
@@
 	(wire
 		(pts
-			(xy 328.93 71.12) (xy 347.98 71.12)
+			(xy 273.05 124.46) (xy 292.1 124.46)
 		)
 		(stroke
@@
 	(wire
 		(pts
-			(xy 328.93 53.34) (xy 328.93 71.12)
+			(xy 273.05 106.68) (xy 273.05 124.46)
 		)
 		(stroke
@@
 	(wire
 		(pts
-			(xy 345.44 68.58) (xy 347.98 68.58)
+			(xy 289.56 121.92) (xy 292.1 121.92)
 		)
 		(stroke
@@
 	(wire
 		(pts
-			(xy 349.25 53.34) (xy 328.93 53.34)
+			(xy 293.37 106.68) (xy 273.05 106.68)
 		)
 		(stroke
@@
 	)
 	(rectangle
-		(start 325.628 45.72)
-		(end 392.43 77.216)
+		(start 269.748 99.06)
+		(end 336.55 130.556)
 		(stroke
 			(width 0.25)
@@
 	(text_box "K12 - Na rectificação de onda completa, \na onda de entrada tem de ser medida primeiro, devido ao problema de massas.\nSendo assim, na primeira medição, K12 estará activo e todos os outros \n11 relés estarão desactivados, é feita a medição.\nPara medir a onda de saída, o relés K12 ficará aberto, cortando, assim, a massa do Canal 1.\nÉ medida a onda de saída e construído o gráfico"
 		(exclude_from_sim no)
-		(at 353.06 81.28 0)
+		(at 525.78 80.01 0)
 		(size 54.102 27.686)
 		(stroke
@@
 		)
 	)
+	(text "Gerador de sinal"
+		(exclude_from_sim no)
+		(at 30.734 72.39 0)
+		(effects
+			(font
+				(size 1.27 1.27)
+			)
+		)
+	)
 	(text "8 relés duplos\n5 relé simples"
 		(exclude_from_sim no)
-		(at 391.668 243.586 0)
+		(at 621.03 97.79 0)
 		(effects
 			(font
@@
 	(text "Relé K12 necessário por causa \ndas massas no rectificador de onda completa"
 		(exclude_from_sim no)
-		(at 44.196 130.302 0)
+		(at -24.13 131.826 0)
 		(effects
 			(font
@@
 		)
 	)
-	(text "Reles simples"
+	(text "Filtragem"
 		(exclude_from_sim no)
-		(at 357.378 41.91 0)
+		(at 301.498 95.25 0)
 		(effects
 			(font
@@
 	(text "Pontas osciloscópio"
 		(exclude_from_sim no)
-		(at 24.384 98.806 0)
+		(at 32.512 90.17 0)
 		(effects
 			(font
@@
 	(text "Total: "
 		(exclude_from_sim no)
-		(at 388.112 234.696 0)
+		(at 617.474 88.9 0)
 		(effects
 			(font
@@
 	(text "Bypass ao díodo para \nrealizar o estudo dos \nfiltros passa-alto e \npassa-baixo\ne resposta do condensador \naos vários tipos de onda"
 		(exclude_from_sim no)
-		(at 326.39 87.122 0)
+		(at 499.11 85.852 0)
 		(effects
 			(font
@@
 	)
 	(label "12V"
-		(at 328.93 49.53 0)
+		(at 273.05 102.87 0)
 		(fields_autoplaced yes)
 		(effects
@@
 	)
 	(label "v_{out}+"
-		(at 374.65 59.69 0)
+		(at 318.77 113.03 0)
 		(fields_autoplaced yes)
 		(effects
@@
 	)
 	(label "O_{24}"
-		(at 364.49 71.12 270)
+		(at 308.61 124.46 270)
 		(fields_autoplaced yes)
 		(effects
@@
 	)
 	(label "O_{23}"
-		(at 365.76 53.34 270)
+		(at 309.88 106.68 270)
 		(fields_autoplaced yes)
 		(effects
@@
 	)
 	(label "v_{in}"
-		(at 345.44 66.04 90)
+		(at 289.56 119.38 90)
 		(fields_autoplaced yes)
 		(effects
@@
 	(symbol
 		(lib_id "Device:R")
-		(at 374.65 54.61 180)
+		(at 318.77 107.95 180)
 		(unit 1)
 		(exclude_from_sim no)
@@
 		(dnp no)
 		(property "Reference" "R3"
-			(at 378.714 55.118 0)
+			(at 322.834 108.458 0)
 			(effects
 				(font
@@
 		)
 		(property "Value" "1K"
-			(at 378.714 53.086 0)
+			(at 322.834 106.426 0)
 			(effects
 				(font
@@
 		)
 		(property "Footprint" "Resistor_THT:R_Axial_DIN0207_L6.3mm_D2.5mm_P15.24mm_Horizontal"
-			(at 376.428 54.61 90)
+			(at 320.548 107.95 90)
 			(effects
 				(font
@@
 		)
 		(property "Datasheet" "~"
-			(at 374.65 54.61 0)
+			(at 318.77 107.95 0)
 			(effects
 				(font
@@
 		)
 		(property "Description" "Resistor"
-			(at 374.65 54.61 0)
+			(at 318.77 107.95 0)
 			(effects
 				(font
@@
 	(symbol
 		(lib_id "3570-1331-123:3570-1331-123")
-		(at 335.915 64.77 0)
+		(at 280.035 118.11 0)
 		(unit 1)
 		(exclude_from_sim no)
@@
 		(dnp no)
 		(property "Reference" "K11"
-			(at 363.22 65.278 0)
+			(at 307.34 118.618 0)
 			(effects
 				(font
@@
 		)
 		(property "Value" "3570-1331-123"
-			(at 356.235 64.77 0)
+			(at 300.355 118.11 0)
 			(effects
 				(font
@@
 		)
 		(property "Footprint" "3570-1331-123:SIP_3570-1331_COM"
-			(at 333.375 57.023 0)
+			(at 277.495 110.363 0)
 			(effects
 				(font
@@
 		)
 		(property "Datasheet" "3570-1331-051"
-			(at 331.343 59.944 0)
+			(at 275.463 113.284 0)
 			(effects
 				(font
@@
 		)
 		(property "Description" ""
-			(at 335.915 64.77 0)
+			(at 280.035 118.11 0)
 			(effects
 				(font
@@
 	(symbol
 		(lib_id "3570-1331-123:3570-1331-123")
-		(at 337.185 46.99 0)
+		(at 281.305 100.33 0)
 		(unit 1)
 		(exclude_from_sim no)
@@
 		(dnp no)
 		(property "Reference" "K10"
-			(at 364.49 47.498 0)
+			(at 308.61 100.838 0)
 			(effects
 				(font
@@
 		)
 		(property "Value" "3570-1331-123"
-			(at 357.505 46.99 0)
+			(at 301.625 100.33 0)
 			(effects
 				(font
@@
 		)
 		(property "Footprint" "3570-1331-123:SIP_3570-1331_COM"
-			(at 334.645 39.243 0)
+			(at 278.765 92.583 0)
 			(effects
 				(font
@@
 		)
 		(property "Datasheet" "3570-1331-051"
-			(at 332.613 42.164 0)
+			(at 276.733 95.504 0)
 			(effects
 				(font
@@
 		)
 		(property "Description" ""
-			(at 337.185 46.99 0)
+			(at 281.305 100.33 0)
 			(effects
 				(font
@@
 	(symbol
 		(lib_id "Device:C_Polarized")
-		(at 374.65 64.77 180)
+		(at 318.77 118.11 180)
 		(unit 1)
 		(exclude_from_sim no)
@@
 		(dnp no)
 		(property "Reference" "C6"
-			(at 373.888 66.802 0)
+			(at 318.008 120.142 0)
 			(effects
 				(font
@@
 		)
 		(property "Value" "10uF"
-			(at 374.396 62.23 0)
+			(at 318.516 115.57 0)
 			(effects
 				(font
@@
 		)
 		(property "Footprint" "Capacitor_THT:CP_Radial_D5.0mm_P2.00mm"
-			(at 373.6848 60.96 0)
+			(at 317.8048 114.3 0)
 			(effects
 				(font
@@
 		)
 		(property "Datasheet" "~"
-			(at 374.65 64.77 0)
+			(at 318.77 118.11 0)
 			(effects
 				(font
@@
 		)
 		(property "Description" "Polarized capacitor"
-			(at 374.65 64.77 0)
+			(at 318.77 118.11 0)
 			(effects
 				(font
