File: disposable_heroes/Kicad_relesSR/meiaonda/meiaonda.kicad_pcb (KiCad board)
At the start: 2 copper layers, 95.2 x 90.2 mm, 28 parts, among them J1 Vgen, J2 Fonte 12V, J3 Fonte 5V - PI5, K1 3572-1220-123, K2 3572-1220-123, K3 3570-1331-123, K4 3572-1220-123, K5 3572-1220-123, K6 3572-1220-123, K7 3572-1220-123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

Commit message: update more circuits
Parts:
- added C5: 10uF, Capacitor_THT:CP_Radial_D6.3mm_P2.50mm, F.Cu at (165.1, 95.2)
- added F1: Fuse, Fuse:Fuseholder_Cylinder-5x20mm_Stelvio-Kontek_PTF78_Horizontal_Open, F.Cu at (97.2, 87.7)
- added J10: Transformer, Connector_PinHeader_2.54mm:PinHeader_1x02_P2.54mm_Vertical, F.Cu at (78.5, 98.5)
- added J4: GPIO11, Connector_PinHeader_2.54mm:PinHeader_1x01_P2.54mm_Vertical, F.Cu at (136.7, 122.0)
- added J5: GPIO26, Connector_PinHeader_2.54mm:PinHeader_1x01_P2.54mm_Vertical, F.Cu at (118.4, 121.9)
- added J6: GPIO6, Connector_PinHeader_2.54mm:PinHeader_1x01_P2.54mm_Vertical, F.Cu at (146.2, 122.0)
- added J7: GPIO13, Connector_PinHeader_2.54mm:PinHeader_1x01_P2.54mm_Vertical, F.Cu at (123.5, 121.9)
- added J8: GPIO5, Connector_PinHeader_2.54mm:PinHeader_1x01_P2.54mm_Vertical, F.Cu at (141.4, 122.0)
- added J9: GND, Connector_PinHeader_2.54mm:PinHeader_1x01_P2.54mm_Vertical, F.Cu at (128.7, 121.8)
- added K10: 3572-1220-123, 3572-1220-123:RELAY8_3572-1220-053_COM, F.Cu at (140.5, 72.3)
- added K11: 3572-1220-123, 3572-1220-123:RELAY8_3572-1220-053_COM, F.Cu at (151.2, 72.2)
- added R3: 1K, Resistor_THT:R_Axial_DIN0207_L6.3mm_D2.5mm_P15.24mm_Horizontal, F.Cu at (136.7, 93.0)
- moved D1 73.6 mm to (90.7, 40.9)
- moved C1 69.7 mm to (143.1, 40.8)
- moved C2 68.1 mm to (152.9, 40.9)
- moved D2 56.9 mm to (111.8, 41.0)
- moved U4 48.3 mm to (147.0, 98.1)
- moved U1 40.9 mm to (88.9, 97.7)
- moved U2 37.2 mm to (108.2, 98.4)
- moved J1 32.7 mm to (78.0, 72.5)
- moved U3 14.8 mm to (128.7, 98.1)
- moved J2 11.5 mm to (78.5, 103.6)
- moved R1 6.86 mm to (77.4, 78.1)
- moved C3 6.07 mm to (77.9, 91.8)
- moved R2 3.35 mm to (77.3, 82.2)
- moved J3 1.65 mm to (78.3, 109.3)
- moved C4 1.21 mm to (78.1, 86.8)
- renumbered K4 to K2, K2 to K3, K3 to K4
Connections:
- net Net-(K2-Pad7) renamed /bypass neg
- K1 pad 1: +12V -> Net-(J1-Pin_1)
- K1 pad 2: Net-(J1-Pin_1) -> +12V
- K1 pad 7: Net-(K1-Pad7) -> /bypass pos
- K2 pad 14: Net-(K1-Pad14) -> Net-(J10-Pin_2)
- K2 pad 8: Net-(K1-Pad7) -> Net-(F1-Pad2)
- K3 pad 8: Net-(K1-Pad7) -> /bypass pos
- K4 pad 4: GND -> Net-(K4-Pad4)
- K5 pad 1: GND -> Net-(K4-Pad4)
- K6 pad 8: GND -> Net-(K4-Pad4)
- K7 pad 8: GND -> Net-(K4-Pad4)
- K8 pad 8: GND -> Net-(K4-Pad4)
- K9 pad 8: GND -> Net-(K4-Pad4)
- U1 pad 10: unconnected-(U1-~SRCLR-Pad10) -> Net-(J5-Pin_1)
- U1 pad 11: unconnected-(U1-SRCLK-Pad11) -> Net-(J7-Pin_1)
- U1 pad 12: unconnected-(U1-RCLK-Pad12) -> Net-(J6-Pin_1)
- U1 pad 13: unconnected-(U1-~OE-Pad13) -> Net-(J4-Pin_1)
- U1 pad 14: unconnected-(U1-SER-Pad14) -> Net-(J8-Pin_1)
- U1 pad 8: unconnected-(U1-GND-Pad8) -> GND
- U2 pad 8: unconnected-(U2-GND-Pad8) -> GND
- U3 pad 1: unconnected-(U3-Q1-Pad1) -> /I_{23}
- U3 pad 10: unconnected-(U3-~SRCLR-Pad10) -> Net-(J5-Pin_1)
- U3 pad 11: unconnected-(U3-SRCLK-Pad11) -> Net-(J7-Pin_1)
- U3 pad 12: unconnected-(U3-RCLK-Pad12) -> Net-(J6-Pin_1)
- U3 pad 13: unconnected-(U3-~OE-Pad13) -> Net-(J4-Pin_1)
- U3 pad 2: unconnected-(U3-Q2-Pad2) -> /I_{24}
- U3 pad 8: unconnected-(U3-GND-Pad8) -> GND
- U4 pad 10: /O_{27} -> unconnected-(U4-O7-Pad10)
- U4 pad 11: /O_{26} -> unconnected-(U4-O6-Pad11)
- U4 pad 8: unconnected-(U4-GND-Pad8) -> GND
Routing:
- net Net-(D1-K): track 98.8 -> 9.65 mm
- net /bypass pos: track 0.00 -> 86.5 mm
- net Net-(D1-A): track 87.6 -> 10.7 mm
- net Net-(K4-Pad4): track 0.00 -> 74.6 mm
- net Net-(J10-Pin_2): track 0.00 -> 74.3 mm
- net Net-(D2-Pad3): track 101.1 -> 27.0 mm
- net /I_{21}: track 36.9 -> 100.9 mm
- net /O_{12}: track 112.3 -> 51.8 mm
- net Net-(C1-Pad2): track 69.8 -> 9.62 mm
- net Net-(J8-Pin_1): track 0.00 -> 59.9 mm
- net Net-(C1-Pad1): track 68.9 -> 9.62 mm, vias 1 -> 0
- net Net-(C2-Pad2): track 68.7 -> 9.80 mm
- net Net-(J4-Pin_1): track 0.00 -> 58.4 mm
- net Net-(J6-Pin_1): track 0.00 -> 58.1 mm
- net GND: track 156.4 -> 101.5 mm
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
Commit message: update kicad
Parts:
- added C6: 10uF, Capacitor_THT:CP_Radial_D5.0mm_P2.00mm, F.Cu at (55.1, 70.8)
- added C_{Out}1: 1uF, Capacitor_THT:CP_Radial_D5.0mm_P2.00mm, F.Cu at (55.1, 77.4)
- added C_{adj}1: 10uF, Capacitor_THT:CP_Radial_D5.0mm_P2.00mm, F.Cu at (55.1, 84.0)
- added C_{i}1: 100nF, Capacitor_THT:C_Disc_D5.1mm_W3.2mm_P5.00mm, F.Cu at (60.9, 84.8)
- added D3: 1N4007, Diode_THT:D_DO-41_SOD81_P10.16mm_Horizontal, F.Cu at (36.2, 77.8)
- added D4: 1N4007, Diode_THT:D_DO-41_SOD81_P10.16mm_Horizontal, F.Cu at (36.2, 82.0)
- added J12: V_{in}, Connector_PinHeader_2.54mm:PinHeader_1x01_P2.54mm_Vertical, F.Cu at (61.9, 62.4)
- added J13: V_{out}, Connector_PinHeader_2.54mm:PinHeader_1x05_P2.54mm_Vertical, F.Cu at (61.6, 69.9)
- added K12: 3570-1331-123, 3570-1331-123:SIP_3570-1331_COM, F.Cu at (37.0, 57.5)
- added K13: 3570-1331-123, 3570-1331-123:SIP_3570-1331_COM, F.Cu at (37.0, 64.2)
- added R4: 330, Resistor_THT:R_Axial_DIN0207_L6.3mm_D2.5mm_P15.24mm_Horizontal, F.Cu at (35.9, 69.6)
- added R5: 1K, Resistor_THT:R_Axial_DIN0207_L6.3mm_D2.5mm_P15.24mm_Horizontal, F.Cu at (35.9, 73.7)
- added T1: Transformer_1P_1S, Connector_PinHeader_2.54mm:PinHeader_1x02_P2.54mm_Vertical, F.Cu at (57.3, 62.4)
- added U5: LM317_TO-220, Package_TO_SOT_THT:TO-220-3_Vertical, F.Cu at (58.2, 58.0)
- J1: value Vgen -> Canal 1 - V_{in}
- J10: value Transformer -> Gerador Sinal
- J4: value GPIO11 -> GPIO22
- J8: value GPIO5 -> GPIO27
- J9: value GND -> Canal 2 - V_{out}; footprint Connector_PinHeader_2.54mm:PinHeader_1x01_P2.54mm_Vertical -> Connector_PinHeader_2.54mm:PinHeader_1x02_P2.54mm_Vertical
- K10, K11: value 3572-1220-123 -> 3570-1331-123; footprint 3572-1220-123:RELAY8_3572-1220-053_COM -> 3570-1331-123:SIP_3570-1331_COM
Connections:
- F1 pad 1: Net-(J10-Pin_1) -> Net-(T1-SB)
- J10 pad 1: Net-(J10-Pin_1) -> Net-(J1-Pin_2)
- J10 pad 2: Net-(J10-Pin_2) -> Net-(J1-Pin_1)
- J9 pad 1: Net-(J9-Pin_1) -> /bypass neg
- K10 pad 1: /bypass neg -> /bypass pos
- K11 pad 1: /bypass neg -> /bypass pos
- K2 pad 1: Net-(D2-Pad3) -> Net-(T1-SA)
- K2 pad 14: Net-(J10-Pin_2) -> Net-(F1-Pad2)
- K2 pad 6: /O_{14} -> /O_{12}
- K2 pad 7: Net-(D2-Pad2) -> Net-(D2-Pad3)
- K2 pad 8: Net-(F1-Pad2) -> Net-(D2-Pad2)
- K3 pad 6: /O_{12} -> /O_{13}
- K4 pad 3: /O_{13} -> /O_{14}
- K4 pad 4: Net-(K4-Pad4) -> Net-(J9-Pin_2)
- K5 pad 1: Net-(K4-Pad4) -> Net-(D2-+)
- K5 pad 8: Net-(D2-+) -> Net-(J9-Pin_2)
- K6 pad 8: Net-(K4-Pad4) -> Net-(J9-Pin_2)
- K7 pad 8: Net-(K4-Pad4) -> Net-(J9-Pin_2)
- K8 pad 8: Net-(K4-Pad4) -> Net-(J9-Pin_2)
- K9 pad 8: Net-(K4-Pad4) -> Net-(J9-Pin_2)
- R3 pad 1: Net-(K10-Pad7) -> /bypass neg
- R3 pad 2: Net-(K10-Pad8) -> Net-(K10-Pad4)
- U2 pad 9: unconnected-(U2-COM-Pad9) -> +12V
- U3 pad 3: unconnected-(U3-Q3-Pad3) -> /I_{25}
- U3 pad 4: unconnected-(U3-Q4-Pad4) -> /I_{26}
- U4 pad 11: unconnected-(U4-O6-Pad11) -> /O_{26}
- U4 pad 9: unconnected-(U4-COM-Pad9) -> +12V
Routing:
- net +12V: track 182.5 -> 0.00 mm
- net GND: track 101.5 -> 0.00 mm
- net /I_{21}: track 100.9 -> 0.00 mm
- net Net-(K7-Pad1): track 94.7 -> 0.00 mm
- net /O_{13}: track 89.9 -> 0.00 mm
- net +5V: track 87.8 -> 0.00 mm
- net /bypass pos: track 86.5 -> 0.00 mm
- net /bypass neg: track 82.2 -> 0.00 mm
- net Net-(K1-Pad14): track 80.1 -> 0.00 mm
- net Net-(K4-Pad4): track 74.6 -> 0.00 mm
- net Net-(J10-Pin_2): track 74.3 -> 0.00 mm
- net Net-(K7-Pad14): track 69.3 -> 0.00 mm, vias 1 -> 0
- net Net-(K6-Pad1): track 63.8 -> 0.00 mm, vias 1 -> 0
- net /O_{11}: track 61.2 -> 0.00 mm
- net Net-(J8-Pin_1): track 59.9 -> 0.00 mm
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- removed copper zone on B.Cu, net GND
- removed copper zone on F.Cu, net GND

Commit message: update - boards done
Parts:
- removed C5: 10uF, Capacitor_THT:CP_Radial_D6.3mm_P2.50mm
- removed C_{Out}1: 1uF, Capacitor_THT:CP_Radial_D5.0mm_P2.00mm
- removed C_{adj}1: 10uF, Capacitor_THT:CP_Radial_D5.0mm_P2.00mm
- removed C_{i}1: 100nF, Capacitor_THT:C_Disc_D5.1mm_W3.2mm_P5.00mm
- removed D3, D4: 1N4007, Diode_THT:D_DO-41_SOD81_P10.16mm_Horizontal
- removed J1: Canal 1 - V_{in}, Connector_PinHeader_2.54mm:PinHeader_1x02_P2.54mm_Vertical
- removed J10: Gerador Sinal, Connector_PinHeader_2.54mm:PinHeader_1x02_P2.54mm_Vertical
- removed J12: V_{in}, Connector_PinHeader_2.54mm:PinHeader_1x01_P2.54mm_Vertical
- removed J13: V_{out}, Connector_PinHeader_2.54mm:PinHeader_1x05_P2.54mm_Vertical
- removed J5: GPIO26, Connector_PinHeader_2.54mm:PinHeader_1x01_P2.54mm_Vertical
- removed J6: GPIO6, Connector_PinHeader_2.54mm:PinHeader_1x01_P2.54mm_Vertical
- removed J7: GPIO13, Connector_PinHeader_2.54mm:PinHeader_1x01_P2.54mm_Vertical
- removed J8: GPIO27, Connector_PinHeader_2.54mm:PinHeader_1x01_P2.54mm_Vertical
- removed J9: Canal 2 - V_{out}, Connector_PinHeader_2.54mm:PinHeader_1x02_P2.54mm_Vertical
- removed R4: 330, Resistor_THT:R_Axial_DIN0207_L6.3mm_D2.5mm_P15.24mm_Horizontal
- removed R5: 1K, Resistor_THT:R_Axial_DIN0207_L6.3mm_D2.5mm_P15.24mm_Horizontal
- removed T1: Transformer_1P_1S, Connector_PinHeader_2.54mm:PinHeader_1x02_P2.54mm_Vertical
- removed U5: LM317_TO-220, Package_TO_SOT_THT:TO-220-3_Vertical
- J2: value Fonte 12V -> PI_config; footprint Connector_PinHeader_2.54mm:PinHeader_1x02_P2.54mm_Vertical -> Connector_PinSocket_2.54mm:PinSocket_1x06_P2.54mm_Vertical
- J3: value Fonte 5V - PI5 -> Power Sources; footprint Connector_PinHeader_2.54mm:PinHeader_1x02_P2.54mm_Vertical -> Connector_PinSocket_2.54mm:PinSocket_1x06_P2.54mm_Vertical
- J4: value GPIO22 -> Signals; footprint Connector_PinHeader_2.54mm:PinHeader_1x01_P2.54mm_Vertical -> Connector_PinSocket_2.54mm:PinSocket_1x06_P2.54mm_Vertical
- moved H2 125.8 mm to (171.3, 125.3)
- moved C6 109.0 mm to (151.5, 121.7), turned to -90 degrees
- moved H4 106.7 mm to (85.5, 47.9)
- moved K13 106.1 mm to (122.7, 126.7), turned to 90 degrees
- moved K12 105.0 mm to (116.0, 126.7), turned to 90 degrees
- moved K4 103.1 mm to (95.8, 126.7), turned to 90 degrees
- moved K1 96.6 mm to (165.2, 89.0)
- moved C2 85.1 mm to (130.4, 122.9)
- moved C1 82.2 mm to (140.8, 122.9)
- moved D2 82.1 mm to (152.2, 112.6), turned to 180 degrees
- moved J2 79.7 mm to (135.4, 47.9), turned to -90 degrees
- moved F1 77.4 mm to (168.3, 57.1), turned to -90 degrees
- moved K3 76.9 mm to (153.6, 88.9)
- moved J4 76.6 mm to (155.9, 47.8), turned to -90 degrees
- moved D1 74.7 mm to (152.5, 82.9)
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Connections:
- net /bypass pos renamed /v_{in}
- C3 pad 1: +5V -> /5V
- C4 pad 1: +5V -> /5V
- C6 pad 2: /bypass neg -> /v_{out}+
- F1 pad 1: Net-(T1-SB) -> /transf+
- J2 pad 1: +12V -> /SRCLK_{filters}
- J2 pad 2: GND -> /~{SRCLR}_{filters}
- J3 pad 1: +5V -> /12V
- J3 pad 2: GND -> /5V
- J4 pad 1: Net-(J4-Pin_1) -> /CH_{1}+
- K1 pad 1: Net-(J1-Pin_1) -> /CH_{1}+
- K1 pad 2: +12V -> /12V
- K1 pad 8: Net-(J1-Pin_2) -> /CH_{1}-
- K10 pad 2: +12V -> /12V
- K11 pad 2: +12V -> /12V
- K12 pad 1: Net-(J1-Pin_2) -> /CH_{1}-
- K12 pad 2: +12V -> /12V
- K13 pad 1: Net-(J1-Pin_1) -> /CH_{1}+
- K13 pad 2: +12V -> /12V
- K2 pad 1: Net-(T1-SA) -> /transf-
- K2 pad 2: +12V -> /12V
- K3 pad 2: +12V -> /12V
- K3 pad 7: /bypass neg -> /v_{out}+
- K4 pad 2: +12V -> /12V
- K4 pad 4: Net-(J9-Pin_2) -> /v_{out}-
- K5 pad 2: +12V -> /12V
- K5 pad 7: /bypass neg -> /v_{out}+
- K5 pad 8: Net-(J9-Pin_2) -> /v_{out}-
- K6 pad 2: +12V -> /12V
- K6 pad 7: /bypass neg -> /v_{out}+
- K6 pad 8: Net-(J9-Pin_2) -> unconnected-(K6-Pad8)
- K7 pad 2: +12V -> /12V
- K7 pad 7: /bypass neg -> /v_{out}+
- K7 pad 8: Net-(J9-Pin_2) -> /v_{out}-
- K8 pad 2: +12V -> /12V
- K8 pad 7: /bypass neg -> /v_{out}+
- K8 pad 8: Net-(J9-Pin_2) -> /v_{out}-
- K9 pad 2: unconnected-(K9-Pad2) -> /12V
- K9 pad 7: /bypass neg -> /v_{out}+
- K9 pad 8: Net-(J9-Pin_2) -> /v_{out}-
- R3 pad 1: /bypass neg -> /v_{out}+
- U1 pad 10: Net-(J5-Pin_1) -> /~{SRCLR}_{filters}
- U1 pad 11: Net-(J7-Pin_1) -> /SRCLK_{filters}
- U1 pad 12: Net-(J6-Pin_1) -> /RCLK_{filters}
- U1 pad 13: Net-(J4-Pin_1) -> /~{OE}_{filters}
- U1 pad 14: Net-(J8-Pin_1) -> /SER_{filters}
- U1 pad 16: +5V -> /5V
- U2 pad 9: +12V -> /12V
- U3 pad 10: Net-(J5-Pin_1) -> /~{SRCLR}_{filters}
- U3 pad 11: Net-(J7-Pin_1) -> /SRCLK_{filters}
- U3 pad 12: Net-(J6-Pin_1) -> /RCLK_{filters}
- U3 pad 13: Net-(J4-Pin_1) -> /~{OE}_{filters}
- U3 pad 16: +5V -> /5V
- U4 pad 9: +12V -> /12V
Routing:
- net /12V: track 0.00 -> 223.9 mm
- net /v_{out}+: track 0.00 -> 163.8 mm
- net /CH_{1}-: track 0.00 -> 143.1 mm
- net /O_{23}: track 0.00 -> 127.4 mm
- net /v_{out}-: track 0.00 -> 124.9 mm
- net /CH_{1}+: track 0.00 -> 119.4 mm
- net Net-(K1-Pad14): track 0.00 -> 104.5 mm
- net GND: track 0.00 -> 104.2 mm
- net /O_{11}: track 0.00 -> 104.2 mm
- net /O_{26}: track 0.00 -> 94.7 mm
- net /O_{13}: track 0.00 -> 87.0 mm
- net /O_{12}: track 0.00 -> 77.6 mm
- net /O_{24}: track 0.00 -> 76.4 mm
- net /v_{in}: track 0.00 -> 75.4 mm
- net Net-(C1-Pad1): track 0.00 -> 74.1 mm
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- added copper zone on B.Cu, net GND
- added copper zone on F.Cu, net GND
Other:
- board size 95.2 x 90.2 mm -> 96 x 90.5 mm
- board text added: "LaRE - Rectifiers and Filters"
