File: disposable_heroes/Kicad_relesSR/power_sources/power_sources.kicad_pcb (KiCad board)
At the start: 2 copper layers, 96 x 90.6 mm, 6 parts

Commit message: update - boards done
Parts:
- added C_{Out}1: 1uF, Capacitor_THT:CP_Radial_D5.0mm_P2.00mm, F.Cu at (112.8, 73.6)
- added C_{adj}1: 10uF, Capacitor_THT:CP_Radial_D5.0mm_P2.00mm, F.Cu at (120.7, 73.7)
- added C_{i}1: 100nF, Capacitor_THT:C_Disc_D5.1mm_W3.2mm_P5.00mm, F.Cu at (127.6, 63.5)
- added D1: 1N4007, Diode_THT:D_DO-41_SOD81_P10.16mm_Horizontal, F.Cu at (133.1, 58.5)
- added D2: 1N4007, Diode_THT:D_DO-41_SOD81_P10.16mm_Horizontal, F.Cu at (143.3, 63.7)
- added J1: V_{in}VB, Connector_PinHeader_2.54mm:PinHeader_1x01_P2.54mm_Vertical, F.Cu at (124.8, 55.6)
- added J2: Transformer, Connector_PinSocket_2.54mm:PinSocket_1x02_P2.54mm_Vertical, F.Cu at (112.0, 55.3)
- added J3: Power Sources, Connector_PinSocket_2.54mm:PinSocket_1x06_P2.54mm_Vertical, F.Cu at (124.7, 47.9)
- added R1: 1K, Resistor_THT:R_Axial_DIN0207_L6.3mm_D2.5mm_P15.24mm_Horizontal, F.Cu at (145.7, 73.6)
- added R2: 330, Resistor_THT:R_Axial_DIN0207_L6.3mm_D2.5mm_P15.24mm_Horizontal, F.Cu at (145.7, 69.0)
- added U1: LM317_TO-220, Package_TO_SOT_THT:TO-220-3_Vertical, F.Cu at (116.1, 62.9)
Routing:
- net /5V: track 0.00 -> 90.2 mm
- net GND: track 0.00 -> 75.7 mm
- net Net-(D2-A): track 0.00 -> 55.9 mm
- net /12V: track 0.00 -> 46.3 mm
- net /transf-: track 0.00 -> 7.49 mm
- net /transf+: track 0.00 -> 7.49 mm
- added copper zone on F.Cu, net GND
Other:
- copper layers 2 -> 4
- board text added: "LaRE - Fonte de tensão"

Commit message: updates finais
Parts:
- added J4: 5V_{VB}, Connector_PinSocket_2.54mm:PinSocket_1x01_P2.54mm_Vertical, F.Cu at (119.7, 55.6)
- J1: footprint Connector_PinHeader_2.54mm:PinHeader_1x01_P2.54mm_Vertical -> Connector_PinSocket_2.54mm:PinSocket_1x01_P2.54mm_Vertical
- moved J2 0.33 mm to (112.0, 55.7)
Routing:
- net /5V_{VB}: track 0.00 -> 7.48 mm
- net /5V: track 90.2 -> 91.5 mm
- net /12V: track 46.3 -> 47.4 mm

Commit message: update kicad files
Parts:
- moved C_{Out}1 63.3 mm to (51.6, 57.2)
- moved C_{adj}1 63.3 mm to (59.5, 57.3)
- moved C_{i}1 63.3 mm to (66.5, 47.1)
- moved H5 63.3 mm to (46.3, 87.1)
- moved R1 63.3 mm to (84.6, 57.2)
- moved H4 63.3 mm to (34.0, 31.5)
- moved J1 63.3 mm to (63.6, 39.2)
- moved J2 63.3 mm to (50.9, 39.3)
- moved J4 63.3 mm to (58.5, 39.2)
- moved D1 63.3 mm to (72.0, 42.1)
- moved D2 63.3 mm to (82.2, 47.3)
- moved H1 63.3 mm to (119.8, 28.9)
- moved H2 63.3 mm to (119.8, 109.0)
- moved H3 63.3 mm to (34.1, 105.2)
- moved H6 63.3 mm to (107.3, 87.1)
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