File: disposable_heroes/Kicad_relesSR/power_sources/power_sources.kicad_sch (KiCad schematic)
At the start: 16 parts, among them J1 V_{in}, J3 Power Sources, U1 LM317_TO-220

Commit message: update - boards done
Parts:
- added J2: Transformer, Connector_PinSocket_2.54mm:PinSocket_1x02_P2.54mm_Vertical, symbol Connector:Conn_01x02_Socket
- J1: value V_{in} -> V_{in}VB; footprint Connector_PinHeader_2.54mm:PinHeader_1x01_P2.54mm_Vertical -> Connector_PinSocket_2.54mm:PinSocket_1x01_P2.54mm_Vertical; symbol Connector:Conn_01x01_Pin -> Connector:Conn_01x01_Socket
- J3: footprint (none) -> Connector_PinSocket_2.54mm:PinSocket_1x06_P2.54mm_Vertical; symbol Connector:Conn_01x04_Socket -> Connector:Conn_01x06_Socket
Connections:
- net 12V: now also C_{i}1.1, D1.1 (K), J1.1 (Pin_1), J3.1 (Pin_1), U1.3 (VI); no longer C_{Out}1.1, D1.2 (A), D2.1 (K), J3.4 (Pin_4), R2.1, U1.2 (VO)
- net 5V: now also C_{Out}1.1, D1.2 (A), D2.1 (K), J3.2 (Pin_2), R2.1, U1.2 (VO); no longer J3.3 (Pin_3)
- net 5V_{VB}: now also J3.3 (Pin_3); no longer J3.2 (Pin_2)
- net GND: now also J3.4 (Pin_4); no longer J3.1 (Pin_1)
- new net transf+: J2.2 (Pin_2), J3.5 (Pin_5)
- new net transf-: J2.1 (Pin_1), J3.6 (Pin_6)
Other:
- moved on the sheet: H1, H2, H3, H4, H5, H6

Commit message: updates finais
Parts:
- added J4: 5V_{VB}, Connector_PinSocket_2.54mm:PinSocket_1x01_P2.54mm_Vertical, symbol Connector:Conn_01x01_Socket
Connections:
- net 5V_{VB}: now also J4.1 (Pin_1)
Changed lines of the file:
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@@
+		)
+	)
+	(symbol
+		(lib_id "Connector:Conn_01x01_Socket")
+		(at 90.17 81.28 90)
+		(unit 1)
+		(exclude_from_sim no)
+		(in_bom yes)
+		(on_board yes)
+		(dnp no)
+		(property "Reference" "J4"
+			(at 91.44 80.6449 90)
+			(effects
+				(font
+					(size 1.27 1.27)
+				)
+				(justify right)
+			)
+		)
+		(property "Value" "5V_{VB}"
+			(at 87.376 80.01 90)
+			(effects
+				(font
+					(size 1.27 1.27)
+				)
+				(justify right)
+			)
+		)
+		(property "Footprint" "Connector_PinSocket_2.54mm:PinSocket_1x01_P2.54mm_Vertical"
+			(at 90.17 81.28 0)
+			(effects
+				(font
+					(size 1.27 1.27)
+				)
+				(hide yes)
+			)
+		)
+		(property "Datasheet" "~"
+			(at 90.17 81.28 0)
+			(effects
+				(font
+					(size 1.27 1.27)
+				)
+				(hide yes)
+			)
+		)
+		(property "Description" "Generic connector, single row, 01x01, script generated"
+			(at 90.17 81.28 0)
+			(effects
+				(font
+					(size 1.27 1.27)
+				)
+				(hide yes)
+			)
+		)
+		(pin "1"
+		)
+		(instances
+			(project "power_sources"
+				(path "/979d2660-1271-462c-82b0-ccec8e0a3ba0"
+					(reference "J4")
+					(unit 1)
+				)
+			)
 		)
 	)

Commit message: update kicad files
Other:
- company: (none) -> ISEP
- title: (none) -> LoRE - Fontes de alimentação
- moved on the sheet: H1, H2, H3, H4, H5, H6
Changed lines of the file:
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@@
 	(generator "eeschema")
 	(generator_version "8.0")
-	(paper "A4")
+	(paper "A4" portrait)
+	(title_block
+		(title "LoRE - Fontes de alimentação")
+		(date "2024-07-20")
+		(rev "Julho 2024")
+		(company "ISEP")
+		(comment 1 "LoRE - Laboratório Remoto Expansível")
+	)
 	(junction
 		(at 69.85 33.02)
@@
 	(symbol
 		(lib_id "Mechanical:MountingHole")
-		(at 250.19 16.51 0)
+		(at 181.61 24.13 0)
 		(unit 1)
 		(exclude_from_sim yes)
@@
 		(fields_autoplaced yes)
 		(property "Reference" "H3"
-			(at 252.73 15.2399 0)
+			(at 184.15 22.8599 0)
 			(effects
 				(font
@@
 		)
 		(property "Value" "MountingHole"
-			(at 252.73 17.7799 0)
+			(at 184.15 25.3999 0)
 			(effects
 				(font
@@
 		)
 		(property "Footprint" "MountingHole:MountingHole_3.2mm_M3"
-			(at 250.19 16.51 0)
+			(at 181.61 24.13 0)
 			(effects
 				(font
@@
 		)
 		(property "Datasheet" "~"
-			(at 250.19 16.51 0)
+			(at 181.61 24.13 0)
 			(effects
 				(font
@@
 		)
 		(property "Description" "Mounting Hole without connection"
-			(at 250.19 16.51 0)
+			(at 181.61 24.13 0)
 			(effects
 				(font
@@
 	(symbol
 		(lib_id "Mechanical:MountingHole")
-		(at 250.19 22.86 0)
+		(at 181.61 30.48 0)
 		(unit 1)
 		(exclude_from_sim yes)
@@
 		(fields_autoplaced yes)
 		(property "Reference" "H4"
-			(at 252.73 21.5899 0)
+			(at 184.15 29.2099 0)
 			(effects
 				(font
@@
 		)
 		(property "Value" "MountingHole"
-			(at 252.73 24.1299 0)
+			(at 184.15 31.7499 0)
 			(effects
 				(font
@@
 		)
 		(property "Footprint" "MountingHole:MountingHole_3.2mm_M3"
-			(at 250.19 22.86 0)
+			(at 181.61 30.48 0)
 			(effects
 				(font
@@
 		)
 		(property "Datasheet" "~"
-			(at 250.19 22.86 0)
+			(at 181.61 30.48 0)
 			(effects
 				(font
@@
 		)
 		(property "Description" "Mounting Hole without connection"
-			(at 250.19 22.86 0)
+			(at 181.61 30.48 0)
 			(effects
 				(font
@@
 	(symbol
 		(lib_id "Mechanical:MountingHole")
-		(at 229.87 29.21 0)
+		(at 161.29 36.83 0)
 		(unit 1)
 		(exclude_from_sim yes)
@@
 		(fields_autoplaced yes)
 		(property "Reference" "H5"
-			(at 232.41 27.9399 0)
+			(at 163.83 35.5599 0)
 			(effects
 				(font
@@
 		)
 		(property "Value" "MountingHole"
-			(at 232.41 30.4799 0)
+			(at 163.83 38.0999 0)
 			(effects
 				(font
@@
 		)
 		(property "Footprint" "MountingHole:MountingHole_3.2mm_M3"
-			(at 229.87 29.21 0)
+			(at 161.29 36.83 0)
 			(effects
 				(font
@@
 		)
 		(property "Datasheet" "~"
-			(at 229.87 29.21 0)
+			(at 161.29 36.83 0)
 			(effects
 				(font
@@
 		)
 		(property "Description" "Mounting Hole without connection"
-			(at 229.87 29.21 0)
+			(at 161.29 36.83 0)
 			(effects
 				(font
@@
 	(symbol
 		(lib_id "Mechanical:MountingHole")
-		(at 229.87 16.51 0)
+		(at 161.29 24.13 0)
 		(unit 1)
 		(exclude_from_sim yes)
@@
 		(fields_autoplaced yes)
 		(property "Reference" "H1"
-			(at 232.41 15.2399 0)
+			(at 163.83 22.8599 0)
 			(effects
 				(font
@@
 		)
 		(property "Value" "MountingHole"
-			(at 232.41 17.7799 0)
+			(at 163.83 25.3999 0)
 			(effects
 				(font
@@
 		)
 		(property "Footprint" "MountingHole:MountingHole_3.2mm_M3"
-			(at 229.87 16.51 0)
+			(at 161.29 24.13 0)
 			(effects
 				(font
@@
 		)
 		(property "Datasheet" "~"
-			(at 229.87 16.51 0)
+			(at 161.29 24.13 0)
 			(effects
 				(font
@@
 		)
 		(property "Description" "Mounting Hole without connection"
-			(at 229.87 16.51 0)
+			(at 161.29 24.13 0)
 			(effects
 				(font
@@
 	(symbol
 		(lib_id "Mechanical:MountingHole")
-		(at 250.19 29.21 0)
+		(at 181.61 36.83 0)
 		(unit 1)
 		(exclude_from_sim yes)
@@
 		(fields_autoplaced yes)
 		(property "Reference" "H6"
-			(at 252.73 27.9399 0)
+			(at 184.15 35.5599 0)
 			(effects
 				(font
@@
 		)
 		(property "Value" "MountingHole"
-			(at 252.73 30.4799 0)
+			(at 184.15 38.0999 0)
 			(effects
 				(font
@@
 		)
 		(property "Footprint" "MountingHole:MountingHole_3.2mm_M3"
-			(at 250.19 29.21 0)
+			(at 181.61 36.83 0)
 			(effects
 				(font
@@
 		)
 		(property "Datasheet" "~"
-			(at 250.19 29.21 0)
+			(at 181.61 36.83 0)
 			(effects
 				(font
@@
 		)
 		(property "Description" "Mounting Hole without connection"
-			(at 250.19 29.21 0)
+			(at 181.61 36.83 0)
 			(effects
 				(font
@@
 	(symbol
 		(lib_id "Mechanical:MountingHole")
-		(at 229.87 22.86 0)
+		(at 161.29 30.48 0)
 		(unit 1)
 		(exclude_from_sim yes)
@@
 		(dnp no)
 		(property "Reference" "H2"
-			(at 232.41 21.5899 0)
+			(at 163.83 29.2099 0)
 			(effects
 				(font
@@
 		)
 		(property "Value" "MountingHole"
-			(at 232.41 24.1299 0)
+			(at 163.83 31.7499 0)
 			(effects
 				(font
@@
 		)
 		(property "Footprint" "MountingHole:MountingHole_3.2mm_M3"
-			(at 229.87 22.86 0)
+			(at 161.29 30.48 0)
 			(effects
 				(font
@@
 		)
 		(property "Datasheet" "~"
-			(at 229.87 22.86 0)
+			(at 161.29 30.48 0)
 			(effects
 				(font
@@
 		)
 		(property "Description" "Mounting Hole without connection"
-			(at 229.87 22.86 0)
-			(effects
-				(font
+			(at 161.29 30.48 0)
+			(effects
+				(font
