File: disposable_heroes/Kicad_relesSR/meiaonda/esquemas_relatorio/esquemas_relatorio.kicad_sch (KiCad schematic)
At the start: 22 parts, among them T1 Transformador 220V/8V, T2 Transformador 220V/8V

Commit message: Finished - uniformização paginas HTML
Parts:
- added C (x4): C_Polarized, symbol Device:C_Polarized
- added MES4, MES5: Osciloscópio, symbol Device:Oscilloscope
- added R10, R7, R8, R9: R, symbol PCM_Elektuur:R
Connections:
- net v_{in}: now also C.1, C.1, C.2, C.2, MES4.1 (-), MES5.1 (-), R10.2 (-), R7.2 (-), R8.2 (-), R9.2 (-)
- new net: C.2, MES5.2 (+), R10.1 (+)
- new net: C.1, R7.1 (+)
- new net: C.2, R9.1 (+)
- new net: C.1, MES4.2 (+), R8.1 (+)

Commit message: update images, diagrams
Parts:
- renumbered Vcc to Ucc
Changed lines of the file:
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@@
 	)
 	(symbol
-		(lib_name "power:AC")
 		(lib_id "power:AC")
 		(at 69.85 121.92 0)
@@
 	)
 	(symbol
-		(lib_name "power:AC")
 		(lib_id "power:AC")
 		(at 31.75 146.05 0)
@@
 	)
 	(symbol
+		(lib_name "vcc:vcc_lare")
 		(lib_id "vcc:vcc_lare")
 		(at 30.48 30.48 0)
@@
 		(on_board yes)
 		(dnp no)
-		(property "Reference" "Vcc"
-			(at 24.13 30.48 0)
+		(property "Reference" "Ucc"
+			(at 23.876 30.48 0)
 			(effects
 				(font
@@
 			(project ""
 				(path "/9fc877dc-cb99-45ed-8cdc-1feaa22a482c"
-					(reference "Vcc")
-					(unit 1)
-				)
-			)
-		)
-	)
-	(symbol
-		(lib_name "power:AC")
+					(reference "Ucc")
+					(unit 1)
+				)
+			)
+		)
+	)
+	(symbol
 		(lib_id "power:AC")
 		(at 69.85 146.05 0)
@@
 	)
 	(symbol
-		(lib_name "power:AC")
 		(lib_id "power:AC")
 		(at 31.75 121.92 0)
